Commit message: can rorate normally

File: urdf/testlx/urdf/testlx.urdf (robot description, URDF)
Before this commit: robot testlx, 2 links, 1 joints
Links:
- link sub: geometry collision box size=2.00000 2.00000 0.55247; visual mesh filename=../meshes/stl/Cube.001.stl scale=1.00000 1.00000 1.00000
Joints:
- joint new_link.000_joint: limit lower=0.00000 upper=0.00000 effort=0.54000 velocity=0.48000 -> lower=0 upper=0 effort=0.54000 velocity=8.70000; origin xyz=-0.07667 2.05628 2.06295 rpy=-0.72994 -0.00000 0.00000 -> xyz=-0.57255 2.22731 0.06915 rpy=-1.57080 0.00000 0.00000; type revolute -> continuous

Commit message: round wheel

File: urdf/testlx/urdf/testlx.urdf (robot description, URDF)
Before this commit: robot testlx, 2 links, 1 joints
Links:
- link sub: geometry collision cylinder length=0.55247 radius=1.00000; visual mesh filename=../meshes/stl/Cube.001.stl scale=1.00000 1.00000 1.00000
Joints:
- joint new_link.000_joint: origin xyz=-0.57255 2.22731 0.06915 rpy=-1.57080 0.00000 0.00000 -> xyz=-0.49588 1.97925 -0.59008 rpy=-1.57080 0.00000 0.00000

Commit message: 3 wheel but no friction

File: urdf/testlx/urdf/testlx.urdf (robot description, URDF)
Before this commit: robot testlx, 2 links, 1 joints
Links:
- added link sub.001, mass 2.46100; collision cylinder length=0.55247 radius=1.00000; visual mesh filename=../meshes/stl/Cube.004.stl scale=1.00000 1.00000 1.00000
- added link sub.002, mass 2.46100; collision cylinder length=0.55247 radius=1.00000; visual mesh filename=../meshes/stl/Cube.020.stl scale=1.00000 1.00000 1.00000
- link myroot: mass None -> 13.89100; geometry collision mesh filename=../meshes/stl/Cube.stl scale=1.00000 1.00000 1.00000; visual mesh filename=../meshes/stl/Cube.stl scale=1.00000 1.00000 1.00000
- link sub: mass None -> 2.46100
Joints:
- removed joint new_link.000_joint
- added joint hw: type continuous, parent myroot, child sub.002, origin xyz=3.49959 0.08915 -0.59008 rpy=-1.57080 0.00000 0.00000, axis 0.00000 0.00000 1.00000, limit lower=0 upper=0 effort=24.09000 velocity=1.26000
- added joint lw: type continuous, parent myroot, child sub.001, origin xyz=-0.49588 -2.24285 -0.59008 rpy=-1.57080 -0.00000 -3.14159, axis 0.00000 0.00000 1.00000, limit lower=0 upper=0 effort=0.54000 velocity=42.30000
- added joint rw: type continuous, parent myroot, child sub, origin xyz=-0.49588 1.97925 -0.59008 rpy=-1.57080 0.00000 0.00000, axis 0.00000 0.00000 1.00000, limit lower=0 upper=0 effort=37.08000 velocity=1.26000

Commit message: .

File: urdf/testlx/urdf/testlx.urdf (robot description, URDF)
Before this commit: robot testlx, 4 links, 3 joints
Links:
- link myroot: geometry visual mesh filename=../meshes/stl/Cube.stl scale=1.00000 1.00000 1.00000
- link sub: geometry collision sphere radius=1.44094; visual mesh filename=../meshes/stl/Cube.001.stl scale=1.00000 1.00000 1.00000
- link sub.001: geometry collision sphere radius=1.44094; visual mesh filename=../meshes/stl/Cube.004.stl scale=1.00000 1.00000 1.00000
- link sub.002: geometry collision sphere radius=1.44094; visual mesh filename=../meshes/stl/Cube.020.stl scale=1.00000 1.00000 1.00000

Commit message: working well finally

File: urdf/testlx/urdf/testlx.urdf (robot description, URDF)
Before this commit: robot testlx, 4 links, 3 joints
Links:
- link sub: geometry collision cylinder length=0.55247 radius=1.00000; visual mesh filename=../meshes/stl/Cube.001.stl scale=1.00000 1.00000 1.00000
- link sub.001: geometry collision cylinder length=0.55247 radius=1.00000; visual mesh filename=../meshes/stl/Cube.004.stl scale=1.00000 1.00000 1.00000
Joints:
- joint hw: limit lower=0 upper=0 effort=24.09000 velocity=1.26000 -> lower=0 upper=0 effort=1000.00000 velocity=1000.00000
- joint lw: limit lower=0 upper=0 effort=0.54000 velocity=42.30000 -> lower=0 upper=0 effort=1000.00000 velocity=1000.00000
- joint rw: limit lower=0 upper=0 effort=37.08000 velocity=1.26000 -> lower=0 upper=0 effort=1000.00000 velocity=1000.00000

Commit message: add camera and global position getter

File: urdf/testlx/urdf/testlx.urdf (robot description, URDF)
Before this commit: robot testlx, 4 links, 3 joints
Links:
- added link end111
- added link new_link
Joints:
- added joint cj: type fixed, parent myroot, child new_link, origin xyz=0.00000 0.00000 0.76100 rpy=0.00000 0.00000 0.00000
- added joint end: type fixed, parent myroot, child end111, origin xyz=-21.22626 1.50564 3.57402 rpy=-1.57080 0.00000 0.00000
